File: irrigation_controller_2/irrigation_controller.kicad_pcb (KiCad board)
At the start: 2 copper layers, 148 x 61 mm, 40 parts, among them J1 Screw_Terminal_01x02, J2 Screw_Terminal_01x02, J3 Screw_Terminal_01x04, J4 Conn_01x04_Pin, J5 Conn_01x04_Pin, Q1 IRL540N, Q2 IRL540N, Q3 IRL540N, Q5 BC547, Q7 BT136-600, U1 XIAO_esp32_C3, U2 FULARR_MP1584EN, U3 MOC3041M

Commit message: modification on label names
Connections:
- net cde_EV1 renamed cmd_EV1
- net cde_EV2 renamed cmd_EV2
- net cde_EV3 renamed cmd_EV3
- net pump_cde renamed pump_cmd
Other:
- board text added: "+3.3V"
- board text added: "GND"
Changed lines of the file:
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@@
 	)
 	(paper "A4")
+	(title_block
+		(title "Irrigation controller - 3 channels")
+		(date "2026-07-13")
+		(rev "1.1")
+		(company "O.Carbonaro")
+		(comment 1 "1.1: minor adjustments on silkscreen")
+	)
 	(layers
 		(0 "F.Cu" signal)
@@
 		(tenting front back)
 		(pcbplotparams
-			(layerselection 0x00000000_00000000_5555555f_575d55f5)
+			(layerselection 0x00000000_00000000_5555555f_575df5f5)
 			(plot_on_all_layers_selection 0x00000000_00000000_00000000_82080021)
 			(disableapertmacros no)
@@
 			(pdf_back_fp_property_popups yes)
 			(pdf_metadata yes)
-			(pdf_single_document yes)
+			(pdf_single_document no)
 			(dxfpolygonmode yes)
 			(dxfimperialunits yes)
@@
 			(psnegative no)
 			(psa4output no)
-			(plot_black_and_white no)
+			(plot_black_and_white yes)
 			(sketchpadsonfab no)
 			(plotpadnumbers no)
@@
 			(crossoutdnponfab yes)
 			(subtractmaskfromsilk no)
-			(outputformat 4)
+			(outputformat 1)
 			(mirror no)
-			(drillshape 2)
+			(drillshape 0)
 			(scaleselection 1)
-			(outputdirectory "")
+			(outputdirectory "./")
 		)
 	)
@@
 	(net 16 "Net-(Q5-B)")
 	(net 17 "Net-(Q7-G)")
-	(net 18 "cde_EV1")
-	(net 19 "cde_EV2")
-	(net 20 "cde_EV3")
+	(net 18 "cmd_EV1")
+	(net 19 "cmd_EV2")
+	(net 20 "cmd_EV3")
 	(net 21 "SW_1")
 	(net 22 "SW_2")
 	(net 23 "SW_3")
 	(net 24 "Net-(U1-GPIO20)")
-	(net 25 "pump_cde")
+	(net 25 "pump_cmd")
 	(net 26 "Net-(R16-Pad2)")
 	(net 27 "Net-(R17-Pad1)")
@@
 			(layers "F.Cu" "F.Mask" "F.Paste")
 			(roundrect_rratio 0.192308)
-			(net 25 "pump_cde")
+			(net 25 "pump_cmd")
 			(pintype "passive")
 		)
@@
 		(tags "connector JST XH vertical")
 		(property "Reference" "J4"
-			(at 9.37 4.95 90)
+			(at 9.37 4.95 0)
 			(layer "F.SilkS")
 			(effects
@@
 		(tags "resistor handsolder")
 		(property "Reference" "R9"
-			(at 3.6 -0.2 0)
+			(at 3.8 0 0)
 			(layer "F.SilkS")
 			(effects
@@
 			(layers "F.Cu" "F.Mask" "F.Paste")
 			(roundrect_rratio 0.192308)
-			(net 19 "cde_EV2")
+			(net 19 "cmd_EV2")
 			(pintype "passive")
 		)
@@
 		(tags "connector JST XH vertical")
 		(property "Reference" "J5"
-			(at -2.08 4.8 270)
+			(at -2.08 4.8 0)
 			(layer "F.SilkS")
 			(effects
@@
 		(tags "resistor handsolder")
 		(property "Reference" "R6"
-			(at 3.7 -1 0)
+			(at 3.8 0.1 0)
 			(layer "F.SilkS")
 			(effects
@@
 			(layers "F.Cu" "F.Mask" "F.Paste")
 			(roundrect_rratio 0.192308)
-			(net 20 "cde_EV3")
+			(net 20 "cmd_EV3")
 			(pintype "passive")
 		)
@@
 		(tags "resistor handsolder")
 		(property "Reference" "R3"
-			(at 3.71 1.21 0)
+			(at 3.8 0 0)
 			(layer "F.SilkS")
 			(effects
@@
 		(tags "resistor handsolder")
 		(property "Reference" "R18"
-			(at -0.12 -2.01 90)
+			(at -0.05 -3 180)
 			(layer "F.SilkS")
 			(effects
@@
 			(layers "*.Cu" "*.Mask")
 			(remove_unused_layers no)
-			(net 18 "cde_EV1")
+			(net 18 "cmd_EV1")
 			(pinfunction "GPIO3")
 			(pintype "bidirectional")
@@
 			(layers "*.Cu" "*.Mask")
 			(remove_unused_layers no)
-			(net 19 "cde_EV2")
+			(net 19 "cmd_EV2")
 			(pinfunction "GPIO4")
 			(pintype "bidirectional")
@@
 			(layers "*.Cu" "*.Mask")
 			(remove_unused_layers no)
-			(net 20 "cde_EV3")
+			(net 20 "cmd_EV3")
 			(pinfunction "GPIO5")
 			(pintype "bidirectional")
@@
 			(layers "*.Cu" "*.Mask")
 			(remove_unused_layers no)
-			(net 25 "pump_cde")
+			(net 25 "pump_cmd")
 			(pinfunction "GPIO6")
 			(pintype "bidirectional")
@@
 			(layers "F.Cu" "F.Mask" "F.Paste")
 			(roundrect_rratio 0.192308)
-			(net 18 "cde_EV1")
+			(net 18 "cmd_EV1")
 			(pintype "passive")
 		)
@@
 	)
 	(gr_text "230V AC"
-		(at 215.1 139.4 0)
+		(at 195.8 139.24 0)
 		(layer "F.SilkS")
 		(effects
@@
 		)
 	)
+	(gr_text "GND"
+		(at 98.1 94.85 0)
+		(layer "F.SilkS")
+		(effects
+			(font
+				(size 0.6 0.6)
+				(thickness 0.1)
+			)
+			(justify left bottom)
+		)
+	)
 	(gr_text "+12V"
 		(at 147.6 131.6 0)
@@
 	)
 	(gr_text "SWITCHS"
-		(at 108.74 93.93 90)
+		(at 108.5 93.6 90)
 		(layer "F.SilkS")
 		(effects
@@
 		)
 	)
+	(gr_text "+3.3V"
+		(at 113 135.9 0)
+		(layer "F.SilkS")
+		(effects
+			(font
+				(size 0.6 0.6)
+				(thickness 0.15)
+			)
+			(justify left bottom)
+		)
+	)
 	(gr_text "O.carbonaro\nV1.0\n07/07/2026"
 		(at 87.9 136.4 0)
@@
 	)
 	(gr_text "pump"
-		(at 194.3 139.1 0)
+		(at 178.7 139.1 0)
 		(layer "F.SilkS")
 		(effects
@@
 	)
 	(gr_text "EV1"
-		(at 145.2 131.9 0)
+		(at 145.2 131.8 0)
 		(layer "B.SilkS")
 		(effects
@@
 	)
 	(gr_text "EV3"
-		(at 135.2 131.7 0)
+		(at 135.2 131.8 0)
 		(layer "B.SilkS")
 		(effects
