File: irrigation_controller_2/irrigation_controller.kicad_sch (KiCad schematic)
At the start: 36 parts, among them J1 Screw_Terminal_01x02, J2 Screw_Terminal_01x02, J3 Screw_Terminal_01x04, J4 Conn_01x04_Pin, J5 Conn_01x04_Pin, Q1 IRL540N, Q2 IRL540N, Q3 IRL540N, Q5 BC547, Q7 BT136-600, U1 XIAO_esp32_C3, U2 FULARR_MP1584EN, U3 MOC3041M

Commit message: modification on label names
Connections:
- net cde_EV1 renamed cmd_EV1
- net cde_EV2 renamed cmd_EV2
- net cde_EV3 renamed cmd_EV3
- net pump_cde renamed pump_cmd
Other:
- note added: "Switchs"
- note removed: "Buttons"
Changed lines of the file:
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@@
 	(title_block
 		(title "Irrigation controller - 3 channels")
-		(date "2026-07-08")
-		(rev "1.0")
+		(date "2026-07-13")
+		(rev "1.1")
 		(company "O.Carbonaro")
-		(comment 1 "0.6: tested design, 3 EVs only")
-		(comment 2 "0.8: SW and LED removed from the board")
-		(comment 3 "0.9: adjustements for pcb routing")
-		(comment 4 "1.0: transfered to production")
+		(comment 1 "0.8: SW and LED removed from the board")
+		(comment 2 "0.9: adjustements for pcb routing")
+		(comment 3 "1.0: transfered to production")
+		(comment 4 "1.1: minor adjustments on label names")
 	)
 	(rectangle
@@
 		)
 	)
-	(text "Buttons "
+	(text "Switchs"
 		(exclude_from_sim no)
 		(at 131.826 145.034 0)
@@
 		)
 	)
-	(global_label "cde_EV1"
+	(global_label "cmd_EV1"
 		(shape input)
 		(at 60.96 43.18 180)
@@
 		)
 		(property "Intersheetrefs" "${INTERSHEET_REFS}"
-			(at 50.2339 43.18 0)
+			(at 49.6292 43.18 0)
 			(effects
 				(font
@@
 		)
 	)
-	(global_label "cde_EV3"
+	(global_label "cmd_EV3"
 		(shape input)
 		(at 60.96 102.87 180)
@@
 		)
 		(property "Intersheetrefs" "${INTERSHEET_REFS}"
-			(at 50.2339 102.87 0)
+			(at 49.6292 102.87 0)
 			(effects
 				(font
@@
 		)
 	)
-	(global_label "cde_EV2"
+	(global_label "cmd_EV2"
 		(shape output)
 		(at 176.53 41.91 180)
@@
 		)
 		(property "Intersheetrefs" "${INTERSHEET_REFS}"
-			(at 165.8039 41.91 0)
+			(at 165.1992 41.91 0)
 			(effects
 				(font
@@
 		)
 	)
-	(global_label "pump_cde"
+	(global_label "pump_cmd"
 		(shape output)
 		(at 176.53 49.53 180)
@@
 		)
 		(property "Intersheetrefs" "${INTERSHEET_REFS}"
-			(at 164.1107 49.53 0)
-			(effects
-				(font
-					(size 1.27 1.27)
-				)
-				(justify right)
-				(hide yes)
-			)
-		)
-	)
-	(global_label "pump_cde"
+			(at 163.506 49.53 0)
+			(effects
+				(font
+					(size 1.27 1.27)
+				)
+				(justify right)
+				(hide yes)
+			)
+		)
+	)
+	(global_label "pump_cmd"
 		(shape input)
 		(at 186.69 110.49 180)
@@
 		)
 		(property "Intersheetrefs" "${INTERSHEET_REFS}"
-			(at 174.2707 110.49 0)
+			(at 173.666 110.49 0)
 			(effects
 				(font
@@
 		)
 	)
-	(global_label "cde_EV3"
+	(global_label "cmd_EV3"
 		(shape output)
 		(at 176.53 45.72 180)
@@
 		)
 		(property "Intersheetrefs" "${INTERSHEET_REFS}"
-			(at 165.8039 45.72 0)
+			(at 165.1992 45.72 0)
 			(effects
 				(font
@@
 		)
 	)
-	(global_label "cde_EV1"
+	(global_label "cmd_EV1"
 		(shape output)
 		(at 176.53 38.1 180)
@@
 		)
 		(property "Intersheetrefs" "${INTERSHEET_REFS}"
-			(at 165.8039 38.1 0)
-			(effects
-				(font
-					(size 1.27 1.27)
-				)
-				(justify right)
-				(hide yes)
-			)
-		)
-	)
-	(global_label "cde_EV2"
+			(at 165.1992 38.1 0)
+			(effects
+				(font
+					(size 1.27 1.27)
+				)
+				(justify right)
+				(hide yes)
+			)
+		)
+	)
+	(global_label "cmd_EV2"
 		(shape input)
 		(at 60.96 72.39 180)
@@
 		)
 		(property "Intersheetrefs" "${INTERSHEET_REFS}"
-			(at 50.2339 72.39 0)
-			(effects
-				(font
+			(at 49.6292 72.39 0)
+			(effects
+				(font
